File: PCB/Kicad/CENTRALE.kicad_pcb (KiCad board)
At the start: 2 copper layers, 100.3 x 72.1 mm, 79 parts, among them IC2 LM358D, J2 RJ11, J3 RJ11, U1 MCP2562-E/SN

Commit message: 2.6.5
Parts:
- renumbered REF** to SMALL_DOWN, REF** to SMALL_SEL, REF to SMALL_UP

Commit message: 2.6.5 II
Other:
- board text added: "c2"
- board text removed: "c1"
Changed lines of the file:
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@@
 		)
 		(property "Value" "50k"
-			(at -2.6935 -4.267757 360)
+			(at -2.6935 -4.267757 0)
 			(layer "F.Fab")
 			(effects
@@
 		)
 	)
-	(gr_text "c1"
+	(gr_text "c2"
 		(at 132.362609 139.7 0)
 		(layer "F.SilkS")

Commit message: PCB c3
Parts:
- removed R19: 15K, CENTRALE02c3:R0805
- removed SJ1, SJ2, SJ4, SJ5: , CENTRALE02c3:SJ
Routing:
- net N$10: track 151.2 -> 143.5 mm
- net N$8: track 41.3 -> 34.2 mm
- net N$39: track 4.07 -> 0.00 mm
- net GND: vias 34 -> 33
Other:
- board text added: "c3"
- board text removed: "c2"

Commit message: PCB 03c4
Parts:
- moved D2 4.82 mm to (152.4, 88.9), turned to -90 degrees
- moved D1 4.64 mm to (157.5, 88.9), turned to -90 degrees
- moved C1 2.19 mm to (156.1, 83.0)
Routing:
- net N$5: track 44.7 -> 58.2 mm
- net N$6: track 55.6 -> 50.0 mm
- net N$18: track 87.6 -> 89.7 mm
- net N$38: track 9.31 -> 10.3 mm
- net N$2: track 9.79 -> 8.79 mm
- net N$1: track 93.4 -> 92.5 mm
- net GND: track 4.10 -> 3.71 mm, vias 33 -> 35
Other:
- board text added: "c4"
- board text removed: "c3"

Commit message: 2.10.0
Parts:
- added BoosterMode1: BoosterInput, Connector_PinHeader_2.54mm:PinHeader_1x05_P2.54mm_Vertical, F.Cu at (124.8, 71.1)
- added REF**: Potentiometer_Bourns_3386C_Horizontal, Potentiometer_THT:Potentiometer_Bourns_3386C_Horizontal, F.Cu at (188.1, 103.2)
- added REF**: - +, Symbol:Symbol_Barrel_Polarity, F.Cu at (188.0, 73.7)
- C1, C10, C11, C12, C13, C2, C3, C4, C5, C8, C9: footprint CENTRALE02c3:C1206 -> Capacitor_SMD:C_1206_3216Metric_Pad1.33x1.80mm_HandSolder
- D1, D2: footprint CENTRALE02c3:SMA-DIODE -> Diode_SMD:D_SOD-128
- L6203: footprint CENTRALE02c3:MULTIWATT-11 -> Package_TO_SOT_THT:TO-220-11_P3.4x5.08mm_StaggerOdd_Lead4.58mm_Vertical
- R10, R12, R15, R18, R20, R21, R3, R4, R5, R6, R7, R8: footprint CENTRALE02c3:R0805 -> Resistor_SMD:R_0805_2012Metric_Pad1.20x1.40mm_HandSolder
- R13, R14: footprint CENTRALE02c3:R2512 -> Resistor_SMD:R_2512_6332Metric_Pad1.40x3.35mm_HandSolder
- R16: footprint CENTRALE02c3:R0805 -> Resistor_SMD:R_0805_2012Metric
- R17: footprint CENTRALE02c3:3386-MULTI -> Potentiometer_THT:Potentiometer_Bourns_3386P_Vertical
- R9: footprint CENTRALE02c3:M1206 -> Resistor_SMD:R_1206_3216Metric_Pad1.30x1.75mm_HandSolder
- moved GOLD_ORB_SM1 55.6 mm to (160.0, 83.8)
- moved L6203 10.2 mm to (152.3, 78.7)
- moved JP5 8.56 mm to (193.0, 88.9)
- moved R17 2.54 mm to (193.2, 103.2), turned to 180 degrees
Connections:
- JP1 pad 11: N$29 -> N$25
- JP1 pad 13: (no net) -> GND
- JP1 pad 7: N$25 -> N$29
- JP1 pad 8: N$26 -> GND
Routing:
- net N$18: track 89.7 -> 137.1 mm
- net N$10: track 143.5 -> 182.0 mm
- net N$34: track 118.3 -> 153.0 mm
- net N$1: track 92.5 -> 119.4 mm
- net N$25: track 5.97 -> 19.3 mm, vias 0 -> 1
- net N$29: track 9.16 -> 19.3 mm
- net N$11: track 54.4 -> 60.9 mm
- net N$5: track 58.2 -> 52.9 mm
- net N$9: track 17.7 -> 18.4 mm, vias 0 -> 1
- net GND: track 3.71 -> 3.84 mm, vias 35 -> 34
Other:
- board text added: "27"
- board text added: "32"
- board text added: "33"
- board text added: "36"
- board text added: "LaBox 1.0"
- board text added: "a1"
- board text removed: "LaBox 0.3"
- board text removed: "c4"

Commit message: 2.10.0 PCB production files
Parts:
- R10, R12, R15, R18, R4, R5, R6, R8: value 10K -> 0805W8F1002T5E
- R13, R14: value 0R5 -> RLP25FEER500
- R16: value 220K -> 0805W8F2203T5E
- R20, R21: value 47K -> 0805W8F4702T5E
- R3: value 33K -> 0805W8F3302T5E
- R7: value 68K -> 0805W8F6802T5E
- R9: value 120R -> 1206W4F1200T5E
Changed lines of the file:
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@@
 			)
 		)
-		(property "Value" "120R"
+		(property "Value" "1206W4F1200T5E"
 			(at 0 -1.83 180)
 			(layer "B.Fab")
+			(hide yes)
 			(effects
 				(font
@@
 			)
 		)
-		(property "Description" ""
+		(property "Description" "120R"
 			(at 0 0 180)
 			(layer "B.Fab")
-			(hide yes)
 			(effects
 				(font
@@
 			)
 		)
-		(property "Value" "33K"
+		(property "Value" "0805W8F3302T5E"
 			(at 0 -1.65 90)
 			(layer "B.Fab")
+			(hide yes)
 			(effects
 				(font
@@
 			)
 		)
-		(property "Description" ""
+		(property "Description" "33K"
 			(at 0 0 90)
 			(layer "B.Fab")
-			(hide yes)
 			(effects
 				(font
@@
 			)
 		)
-		(property "Value" "47K"
+		(property "Value" "0805W8F4702T5E"
 			(at 0 -1.65 90)
 			(layer "B.Fab")
+			(hide yes)
 			(effects
 				(font
@@
 			)
 		)
-		(property "Description" ""
+		(property "Description" "47K"
 			(at 0 0 90)
 			(layer "B.Fab")
-			(hide yes)
 			(effects
 				(font
@@
 			)
 		)
-		(property "Value" "10K"
+		(property "Value" "0805W8F1002T5E"
 			(at 0 -1.65 0)
 			(layer "B.Fab")
@@
 			)
 		)
-		(property "Description" ""
+		(property "Description" "10K"
 			(at 0 0 0)
 			(layer "B.Fab")
@@
 			)
 		)
-		(property "Value" "0R5"
+		(property "Value" "RLP25FEER500"
 			(at 0 -2.63 270)
 			(layer "B.Fab")
+			(hide yes)
 			(effects
 				(font
@@
 			)
 		)
-		(property "Description" ""
+		(property "Description" "0R5"
 			(at 0 0 270)
 			(layer "B.Fab")
-			(hide yes)
 			(effects
 				(font
@@
 			)
 		)
-		(property "Value" "10K"
+		(property "Value" "0805W8F1002T5E"
 			(at 0 -1.65 270)
 			(layer "B.Fab")
+			(hide yes)
 			(effects
 				(font
@@
 			)
 		)
-		(property "Description" ""
+		(property "Description" "10K"
 			(at 0 0 270)
 			(layer "B.Fab")
-			(hide yes)
 			(effects
 				(font
@@
 			)
 		)
-		(property "Value" "47K"
+		(property "Value" "0805W8F4702T5E"
 			(at 0 -1.65 90)
 			(layer "B.Fab")
@@
 			)
 		)
-		(property "Description" ""
+		(property "Description" "47K"
 			(at 0 0 90)
 			(layer "B.Fab")
@@
 			)
 		)
+		(property "FT Rotation Offset" "180"
+			(at 0 0 0)
+			(unlocked yes)
+			(layer "B.Fab")
+			(hide yes)
+			(effects
+				(font
+					(size 1 1)
+					(thickness 0.15)
+				)
+				(justify mirror)
+			)
+		)
 		(attr smd)
 		(fp_line
@@
 			)
 		)
-		(property "Value" "10K"
+		(property "Value" "0805W8F1002T5E"
 			(at 0 -1.65 270)
 			(layer "B.Fab")
@@
 			)
 		)
-		(property "Description" ""
+		(property "Description" "10K"
 			(at 0 0 270)
 			(layer "B.Fab")
@@
 			)
 		)
+		(property "FT Rotation Offset" "-90"
+			(at 0 0 0)
+			(unlocked yes)
+			(layer "B.Fab")
+			(hide yes)
+			(effects
+				(font
+					(size 1 1)
+					(thickness 0.15)
+				)
+				(justify mirror)
+			)
+		)
 		(attr smd)
 		(fp_line
@@
 			)
 		)
-		(property "Value" "0R5"
+		(property "Value" "RLP25FEER500"
 			(at 0 -2.63 270)
 			(layer "B.Fab")
+			(hide yes)
 			(effects
 				(font
@@
 			)
 		)
-		(property "Description" ""
+		(property "Description" "0R5"
 			(at 0 0 270)
 			(layer "B.Fab")
-			(hide yes)
 			(effects
 				(font
@@
 			)
 		)
+		(property "FT Rotation Offset" "0"
+			(at 0 0 0)
+			(unlocked yes)
+			(layer "B.Fab")
+			(hide yes)
+			(effects
+				(font
+					(size 1 1)
+					(thickness 0.15)
+				)
+				(justify mirror)
+			)
+		)
 		(attr smd)
 		(fp_line
@@
 			)
 		)
-		(property "Value" "10K"
+		(property "Value" "0805W8F1002T5E"
 			(at 3.345677 0.014627 0)
 			(layer "B.Fab")
@@
 			)
 		)
-		(property "Description" ""
+		(property "Description" "10K"
 			(at 0 0 0)
 			(layer "B.Fab")
@@
 			)
 		)
-		(property "Value" "10K"
+		(property "Value" "0805W8F1002T5E"
 			(at 0 -1.65 180)
 			(layer "B.Fab")
+			(hide yes)
 			(effects
 				(font
@@
 			)
 		)
-		(property "Description" ""
-			(at 0 0 180)
+		(property "Description" "10K"
+			(at -3.659993 0.668616 180)
 			(layer "B.Fab")
-			(hide yes)
 			(effects
 				(font
@@
 			)
 		)
+		(property "FT Rotation Offset" "180"
+			(at 0 0 0)
+			(unlocked yes)
+			(layer "B.Fab")
+			(hide yes)
+			(effects
+				(font
+					(size 1 1)
+					(thickness 0.15)
+				)
+				(justify mirror)
+			)
+		)
 		(fp_line
 			(start 2.165 -1.28)
@@
 			)
 		)
-		(property "Value" "10K"
+		(property "Value" "0805W8F1002T5E"
 			(at 0 -1.65 0)
 			(layer "B.Fab")
+			(hide yes)
 			(effects
 				(font
@@
 			)
 		)
-		(property "Description" ""
+		(property "Description" "10K"
 			(at 0 0 0)
 			(layer "B.Fab")
-			(hide yes)
 			(effects
 				(font
@@
 			)
 		)
+		(property "FT Rotation Offset" "180"
+			(at 0 0 0)
+			(unlocked yes)
+			(layer "B.Fab")
+			(hide yes)
+			(effects
+				(font
+					(size 1 1)
+					(thickness 0.15)
+				)
+				(justify mirror)
+			)
+		)
 		(attr smd)
 		(fp_line
@@
 			)
 		)
-		(property "Value" "10K"
+		(property "Value" "0805W8F1002T5E"
 			(at 3.435605 0.11912 180)
 			(layer "B.Fab")
+			(hide yes)
 			(effects
 				(font
@@
 			)
 		)
-		(property "Description" ""
+		(property "Description" "10K"
 			(at 0 0 180)
 			(layer "B.Fab")
-			(hide yes)
 			(effects
 				(font
@@
 			)
 		)
-		(property "Value" "10K"
+		(property "Value" "0805W8F1002T5E"
 			(at 0 -1.65 90)
 			(layer "B.Fab")
@@
 			)
 		)
-		(property "Description" ""
+		(property "Description" "10K"
 			(at 0 0 90)
 			(layer "B.Fab")
@@
 			)
 		)
-		(property "Value" "68K"
+		(property "Value" "0805W8F6802T5E"
 			(at 0 -1.65 0)
 			(layer "B.Fab")
+			(hide yes)
 			(effects
 				(font
@@
 			)
 		)
-		(property "Description" ""
-			(at 0 0 0)
+		(property "Description" "68K"
+			(at 0 -1.951259 0)
 			(layer "B.Fab")
-			(hide yes)
 			(effects
 				(font
@@
 			)
 		)
-		(property "Value" "220K"
+		(property "Value" "0805W8F2203T5E"
 			(at 0 -1.65 270)
 			(layer "B.Fab")
+			(hide yes)
 			(effects
 				(font
@@
 			)
 		)
-		(property "Description" ""
+		(property "Description" "220K"
 			(at 0 0 270)
 			(layer "B.Fab")
-			(hide yes)
 			(effects
 				(font
@@
 		(min_thickness 0.25)
 		(filled_areas_thickness no)
-		(fill
+		(fill yes
 			(thermal_gap 0.5)
 			(thermal_bridge_width 0.5)
@@
 		(min_thickness 0.25)
 		(filled_areas_thickness no)
-		(fill
+		(fill yes
 			(thermal_gap 0.5)
 			(thermal_bridge_width 0.5)

Commit message: 2.10.0 PCB Production files II
Parts:
- U$1: value DC-DC-STEP-DOWNDC-DC -> DC-DC-STEP-DOWN
Other:
- board text added: "a2"
- board text removed: "a1"

Commit message: PCB 1.0a2
Other:
- board text added: "1"
Changed lines of the file:
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@@
 			)
 		)
-		(attr through_hole)
+		(attr through_hole exclude_from_pos_files exclude_from_bom dnp)
 		(fp_line
 			(start 4.86 -7.415)
@@
 			)
 		)
-		(attr through_hole)
+		(attr through_hole exclude_from_pos_files exclude_from_bom dnp)
 		(fp_line
 			(start -2.525 -2.335)
@@
 			)
 		)
-		(attr through_hole)
+		(attr through_hole exclude_from_pos_files exclude_from_bom dnp)
 		(fp_line
 			(start -1.72 -9.7)
@@
 			)
 		)
-		(attr through_hole)
+		(attr through_hole exclude_from_pos_files exclude_from_bom dnp)
 		(fp_line
 			(start -1.38 -1.38)
@@
 	)
 	(gr_line
+		(start 157.512532 89.197875)
+		(end 157.118075 89.197875)
+		(stroke
+			(width 0.12)
+			(type default)
+		)
+		(layer "B.SilkS")
+	)
+	(gr_line
+		(start 187.065118 75.997167)
+		(end 187.065118 75.507146)
+		(stroke
+			(width 0.12)
+			(type default)
+		)
+		(layer "B.SilkS")
+	)
+	(gr_line
+		(start 152.4 89.15416)
+		(end 152.794072 89.158226)
+		(stroke
+			(width 0.12)
+			(type default)
+		)
+		(layer "B.SilkS")
+	)
+	(gr_line
+		(start 187.453836 75.4985)
+		(end 187.065118 74.870717)
+		(stroke
+			(width 0.12)
+			(type default)
+		)
+		(layer "B.SilkS")
+	)
+	(gr_line
+		(start 152.4 89.648247)
+		(end 152.4 89.158226)
+		(stroke
+			(width 0.12)
+			(type default)
+		)
+		(layer "B.SilkS")
+	)
+	(gr_line
+		(start 152.788718 89.14958)
+		(end 152.4 88.521797)
+		(stroke
+			(width 0.12)
+			(type default)
+		)
+		(layer "B.SilkS")
+	)
+	(gr_line
+		(start 157.118075 89.197875)
+		(end 157.512532 88.602124)
+		(stroke
+			(width 0.12)
+			(type default)
+		)
+		(layer "B.SilkS")
+	)
+	(gr_line
+		(start 158.022059 88.561446)
+		(end 157.003004 88.561446)
+		(stroke
+			(width 0.12)
+			(type default)
+		)
+		(layer "B.SilkS")
+	)
+	(gr_line
+		(start 157.512532 89.193809)
+		(end 157.906604 89.197875)
+		(stroke
+			(width 0.12)
+			(type default)
+		)
+		(layer "B.SilkS")
+	)
+	(gr_line
+		(start 152.005543 89.158226)
+		(end 152.4 88.562475)
+		(stroke
+			(width 0.12)
+			(type default)
+		)
+		(layer "B.SilkS")
+	)
+	(gr_line
+		(start 186.670661 75.507146)
+		(end 187.065118 74.911395)
+		(stroke
+			(width 0.12)
+			(type default)
+		)
+		(layer "B.SilkS")
+	)
+	(gr_line
+		(start 152.4 88.521797)
+		(end 152.4 88.01227)
+		(stroke
+			(width 0.12)
+			(type default)
+		)
+		(layer "B.SilkS")
+	)
+	(gr_line
+		(start 157.90125 89.189229)
+		(end 157.512532 88.561446)
+		(stroke
+			(width 0.12)
+			(type default)
+		)
+		(layer "B.SilkS")
+	)
+	(gr_line
+		(start 187.065118 75.50308)
+		(end 187.45919 75.507146)
+		(stroke
+			(width 0.12)
+			(type default)
+		)
+		(layer "B.SilkS")
+	)
+	(gr_line
+		(start 187.065118 75.507146)
+		(end 186.670661 75.507146)
+		(stroke
+			(width 0.12)
+			(type default)
+		)
+		(layer "B.SilkS")
+	)
+	(gr_line
+		(start 157.512532 88.561446)
+		(end 157.512532 88.051919)
+		(stroke
+			(width 0.12)
+			(type default)
+		)
+		(layer "B.SilkS")
+	)
+	(gr_line
+		(start 187.574645 74.870717)
+		(end 186.55559 74.870717)
+		(stroke
+			(width 0.12)
+			(type default)
+		)
+		(layer "B.SilkS")
+	)
+	(gr_line
+		(start 152.909527 88.521797)
+		(end 151.890472 88.521797)
+		(stroke
+			(width 0.12)
+			(type default)
+		)
+		(layer "B.SilkS")
+	)
+	(gr_line
+		(start 152.4 89.158226)
+		(end 152.005543 89.158226)
+		(stroke
+			(width 0.12)
+			(type default)
+		)
+		(layer "B.SilkS")
+	)
+	(gr_line
+		(start 187.065118 74.870717)
+		(end 187.065118 74.36119)
+		(stroke
+			(width 0.12)
+			(type default)
+		)
+		(layer "B.SilkS")
+	)
+	(gr_line
+		(start 157.512532 89.687896)
+		(end 157.512532 89.197875)
+		(stroke
+			(width 0.12)
+			(type default)
+		)
+		(layer "B.SilkS")
+	)
+	(gr_line
 		(start 198.6661 140.57)
 		(end 198.6661 68.434)
@@
 		)
 	)
+	(gr_text "1"
+		(at 178.664652 107.43657 0)
+		(layer "B.SilkS")
+		(effects
+			(font
+				(size 1 1)
+				(thickness 0.15)
+			)
+			(justify left bottom mirror)
+		)
+	)
+	(gr_text "1"
+		(at 114.917608 103.946638 0)
+		(layer "B.SilkS")
+		(effects
+			(font
+				(size 1 1)
+				(thickness 0.15)
+			)
+			(justify left bottom mirror)
+		)
+	)
 	(segment
 		(start 104.816443 117.71)
@@
 	)
 	(via
-		(at 114.437179 102.217743)
+		(at 115.158514 102.447713)
 		(size 0.7564)
 		(drill 0.35)
@@
 	)
 	(via
-		(at 157.48 88.9)
+		(at 161.3888 87.54126)
 		(size 0.7564)
 		(drill 0.35)
