File: PCB/Kicad/CENTRALE.kicad_pcb (KiCad board)
At the start: 2 copper layers, 100.3 x 72.1 mm, 77 parts, among them IC2 LM358D, J2 RJ11, J3 RJ11, U1 MCP2562-E/SN

Commit message: PCB 1.0a3
Parts:
- D1, D2: footprint Diode_SMD:D_SOD-128 -> Diode_SMD:D_SOD-123
Connections:
- D1 pad 1: (no net) -> GND
- D2 pad 1: (no net) -> GND
Routing:
- net GND: vias 34 -> 39
Other:
- board text added: "a3"
- board text removed: "a2"
Changed lines of the file:
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@@
 		(property "Value" "-       +"
 			(at 0 0 90)
-			(layer "F.Fab")
+			(layer "F.SilkS")
 			(effects
 				(font
@@
 		)
 	)
-	(footprint "Diode_SMD:D_SOD-128"
+	(footprint "Diode_SMD:D_SOD-123"
 		(layer "B.Cu")
 		(at 152.4 88.9 -90)
-		(descr "D_SOD-128 (CFP5 SlimSMAW), https://assets.nexperia.com/documents/outline-drawing/SOD128.pdf")
-		(tags "D_SOD-128")
+		(descr "SOD-123")
+		(tags "SOD-123")
 		(property "Reference" "D2"
-			(at 4.123433 -0.077468 0)
+			(at 3.207536 0.027447 0)
 			(layer "B.SilkS")
 			(effects
@@
 		)
 		(property "Value" "1N5819"
-			(at 0 2.493967 90)
+			(at 0 -2.1 90)
 			(layer "B.Fab")
 			(effects
@@
 		(attr smd)
 		(fp_line
-			(start -3.16 1.36)
-			(end 1.9 1.36)
+			(start -2.36 1)
+			(end 1.65 1)
 			(stroke
 				(width 0.12)
@@
 		)
 		(fp_line
-			(start -3.16 1.36)
-			(end -3.16 -1.36)
+			(start -2.36 1)
+			(end -2.36 -1)
 			(stroke
 				(width 0.12)
@@
 		)
 		(fp_line
-			(start -3.16 -1.36)
-			(end 1.9 -1.36)
+			(start -2.36 -1)
+			(end 1.65 -1)
 			(stroke
 				(width 0.12)
@@
 		)
 		(fp_line
-			(start -3.15 1.5)
-			(end 3.15 1.5)
+			(start -2.35 1.15)
+			(end 2.35 1.15)
 			(stroke
 				(width 0.05)
@@
 		)
 		(fp_line
-			(start -3.15 1.5)
-			(end -3.15 -1.5)
+			(start -2.35 1.15)
+			(end -2.35 -1.15)
 			(stroke
 				(width 0.05)
@@
 		)
 		(fp_line
-			(start 3.15 1.5)
-			(end 3.15 -1.5)
+			(start 2.35 1.15)
+			(end 2.35 -1.15)
 			(stroke
 				(width 0.05)
@@
 		)
 		(fp_line
-			(start 3.15 -1.5)
-			(end -3.15 -1.5)
+			(start 2.35 -1.15)
+			(end -2.35 -1.15)
 			(stroke
 				(width 0.05)
@@
 		)
 		(fp_line
-			(start -1.9 1.25)
-			(end 1.9 1.25)
+			(start -1.4 0.9)
+			(end 1.4 0.9)
 			(stroke
 				(width 0.1)
@@
 		)
 		(fp_line
-			(start 1.9 1.25)
-			(end 1.9 -1.25)
+			(start 1.4 0.9)
+			(end 1.4 -0.9)
 			(stroke
 				(width 0.1)
@@
 		)
 		(fp_line
-			(start -1.9 -1.25)
-			(end -1.9 1.25)
+			(start -1.4 -0.9)
+			(end -1.4 0.9)
 			(stroke
 				(width 0.1)
@@
 		)
 		(fp_line
-			(start 1.9 -1.25)
-			(end -1.9 -1.25)
+			(start 1.4 -0.9)
+			(end -1.4 -0.9)
 			(stroke
 				(width 0.1)
@@
 			(layer "B.Fab")
 		)
+		(fp_text user "${REFERENCE}"
+			(at 0 2 90)
+			(layer "B.Fab")
+			(effects
+				(font
+					(size 1 1)
+					(thickness 0.15)
+				)
+				(justify mirror)
+			)
+		)
 		(pad "1" smd roundrect
-			(at -2.2 0 270)
-			(size 1.4 2.1)
+			(at -1.65 0 270)
+			(size 0.9 1.2)
 			(layers "B.Cu" "B.Mask" "B.Paste")
-			(roundrect_rratio 0.1785714286)
+			(roundrect_rratio 0.25)
+			(net 7 "GND")
 		)
 		(pad "2" smd roundrect
-			(at 2.2 0 270)
-			(size 1.4 2.1)
+			(at 1.65 0 270)
+			(size 0.9 1.2)
 			(layers "B.Cu" "B.Mask" "B.Paste")
-			(roundrect_rratio 0.1785714286)
+			(roundrect_rratio 0.25)
 		)
 		(embedded_fonts no)
-		(model "${KICAD9_3DMODEL_DIR}/Diode_SMD.3dshapes/D_SOD-128.wrl"
+		(model "${KICAD9_3DMODEL_DIR}/Diode_SMD.3dshapes/D_SOD-123.wrl"
 			(offset
 				(xyz 0 0 0)
@@
 		)
 	)
-	(footprint "Diode_SMD:D_SOD-128"
+	(footprint "Diode_SMD:D_SOD-123"
 		(layer "B.Cu")
 		(at 157.48 88.9 -90)
-		(descr "D_SOD-128 (CFP5 SlimSMAW), https://assets.nexperia.com/documents/outline-drawing/SOD128.pdf")
-		(tags "D_SOD-128")
+		(descr "SOD-123")
+		(tags "SOD-123")
 		(property "Reference" "D1"
-			(at 4.123433 0.116509 0)
+			(at 3.181861 0.049578 0)
 			(layer "B.SilkS")
 			(effects
@@
 		)
 		(property "Value" "1N5819"
-			(at -1.667069 -2.490422 90)
+			(at 0 -2.1 90)
 			(layer "B.Fab")
 			(effects
@@
 		(attr smd)
 		(fp_line
-			(start -3.16 1.36)
-			(end 1.9 1.36)
+			(start -2.36 1)
+			(end 1.65 1)
 			(stroke
 				(width 0.12)
@@
 		)
 		(fp_line
-			(start -3.16 1.36)
-			(end -3.16 -1.36)
+			(start -2.36 1)
+			(end -2.36 -1)
 			(stroke
 				(width 0.12)
@@
 		)
 		(fp_line
-			(start -3.16 -1.36)
-			(end 1.9 -1.36)
+			(start -2.36 -1)
+			(end 1.65 -1)
 			(stroke
 				(width 0.12)
@@
 		)
 		(fp_line
-			(start -3.15 1.5)
-			(end 3.15 1.5)
+			(start -2.35 1.15)
+			(end 2.35 1.15)
 			(stroke
 				(width 0.05)
@@
 		)
 		(fp_line
-			(start -3.15 1.5)
-			(end -3.15 -1.5)
+			(start -2.35 1.15)
+			(end -2.35 -1.15)
 			(stroke
 				(width 0.05)
@@
 		)
 		(fp_line
-			(start 3.15 1.5)
-			(end 3.15 -1.5)
+			(start 2.35 1.15)
+			(end 2.35 -1.15)
 			(stroke
 				(width 0.05)
@@
 		)
 		(fp_line
-			(start 3.15 -1.5)
-			(end -3.15 -1.5)
+			(start 2.35 -1.15)
+			(end -2.35 -1.15)
 			(stroke
 				(width 0.05)
@@
 		)
 		(fp_line
-			(start -1.9 1.25)
-			(end 1.9 1.25)
+			(start -1.4 0.9)
+			(end 1.4 0.9)
 			(stroke
 				(width 0.1)
@@
 		)
 		(fp_line
-			(start 1.9 1.25)
-			(end 1.9 -1.25)
+			(start 1.4 0.9)
+			(end 1.4 -0.9)
 			(stroke
 				(width 0.1)
@@
 		)
 		(fp_line
-			(start -1.9 -1.25)
-			(end -1.9 1.25)
+			(start -1.4 -0.9)
+			(end -1.4 0.9)
 			(stroke
 				(width 0.1)
@@
 		)
 		(fp_line
-			(start 1.9 -1.25)
-			(end -1.9 -1.25)
+			(start 1.4 -0.9)
+			(end -1.4 -0.9)
 			(stroke
 				(width 0.1)
@@
 			(layer "B.Fab")
 		)
+		(fp_text user "${REFERENCE}"
+			(at 0 2 90)
+			(layer "B.Fab")
+			(effects
+				(font
+					(size 1 1)
+					(thickness 0.15)
+				)
+				(justify mirror)
+			)
+		)
 		(pad "1" smd roundrect
-			(at -2.2 0 270)
-			(size 1.4 2.1)
+			(at -1.65 0 270)
+			(size 0.9 1.2)
 			(layers "B.Cu" "B.Mask" "B.Paste")
-			(roundrect_rratio 0.1785714286)
+			(roundrect_rratio 0.25)
+			(net 7 "GND")
 		)
 		(pad "2" smd roundrect
-			(at 2.2 0 270)
-			(size 1.4 2.1)
+			(at 1.65 0 270)
+			(size 0.9 1.2)
 			(layers "B.Cu" "B.Mask" "B.Paste")
-			(roundrect_rratio 0.1785714286)
+			(roundrect_rratio 0.25)
 		)
 		(embedded_fonts no)
-		(model "${KICAD9_3DMODEL_DIR}/Diode_SMD.3dshapes/D_SOD-128.wrl"
+		(model "${KICAD9_3DMODEL_DIR}/Diode_SMD.3dshapes/D_SOD-123.wrl"
 			(offset
 				(xyz 0 0 0)
@@
 		)
 	)
-	(gr_text "a2"
+	(gr_text "a3"
 		(at 127.899742 140.219907 0)
 		(layer "F.SilkS")
@@
 	)
 	(via
-		(at 165.1 93.98)
+		(at 167.64 96.52)
 		(size 0.7564)
 		(drill 0.35)
@@
 	)
 	(via
-		(at 117.5 113)
+		(at 129.237221 105.8581)
 		(size 0.7564)
 		(drill 0.35)
@@
 	)
 	(via
-		(at 154.5 114)
+		(at 157.257487 109.853303)
+		(size 0.7564)
+		(drill 0.35)
+		(layers "F.Cu" "B.Cu")
+		(net 7)
+	)
+	(via
+		(at 166.005693 75.146443)
+		(size 0.7564)
+		(drill 0.35)
+		(layers "F.Cu" "B.Cu")
+		(net 7)
+	)
+	(via
+		(at 134.4363 112.643997)
 		(size 0.7564)
 		(drill 0.35)
@@
 	)
 	(via
-		(at 152.4 83.82)
+		(at 149.86 73.66)
 		(size 0.7564)
 		(drill 0.35)
@@
 	)
 	(via
+		(at 170.781143 81.873153)
+		(size 0.7564)
+		(drill 0.35)
+		(layers "F.Cu" "B.Cu")
+		(net 7)
+	)
+	(via
 		(at 142.44554 112.537155)
 		(size 0.7564)
@@
 	)
 	(via
+		(at 122.879014 80.73883)
+		(size 0.7564)
+		(drill 0.35)
+		(layers "F.Cu" "B.Cu")
+		(net 7)
+	)
+	(via
 		(at 156 101.6)
 		(size 0.7564)
 		(drill 0.35)
+		(layers "F.Cu" "B.Cu")
+		(net 7)
+	)
+	(via
+		(at 157.329731 95.576229)
+		(size 0.7564)
+		(drill 0.35)

Commit message: PCB 1.0a4
Parts:
- D1, D2: value 1N5819 -> K1N5819HW-7-F
Other:
- board text added: "a4"
- board text removed: "a3"
Changed lines of the file:
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@@
 		(tags "TO-220-11 Vertical RM 1.7mm Multiwatt-11 staggered type-1")
 		(property "Reference" "L6203"
-			(at 8.5 -10.7 0)
+			(at 8.465586 -6.966597 0)
 			(layer "F.SilkS")
 			(effects
@@
 			)
 		)
-		(property "Value" "1N5819"
+		(property "Value" " K1N5819HW-7-F"
 			(at 0 -2.1 90)
 			(layer "B.Fab")
@@
 			)
 		)
-		(property "Value" "1N5819"
+		(property "Value" " K1N5819HW-7-F"
 			(at 0 -2.1 90)
 			(layer "B.Fab")
@@
 		(layer "B.SilkS")
 	)
+	(gr_rect
+		(start 177.632681 102.899)
+		(end 180.302825 107.571753)
+		(stroke
+			(width 0.2)
+			(type solid)
+		)
+		(fill no)
+		(layer "B.SilkS")
+	)
 	(gr_line
 		(start 157.512532 89.193809)
@@
 		)
 	)
-	(gr_text "a3"
+	(gr_text "a4"
 		(at 127.899742 140.219907 0)
 		(layer "F.SilkS")

Commit message: PCB 1.0a5 II
Connections:
- D1 pad 2: (no net) -> N$5
- D2 pad 2: (no net) -> N$6
- R17 pad 2: 3V3 -> (no net)
- REF** pad 1: (no net) -> N$35
- REF** pad 2: (no net) -> 3V3
- REF** pad 3: (no net) -> 3V3
Routing:
- net VS: track 102.4 -> 96.8 mm
- net N$9: vias 1 -> 0
- net GND: vias 39 -> 40
Other:
- board text added: "+ +"
- board text added: "a5"
- board text removed: "a4"
Changed lines of the file:
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@@
 			(layers "*.Cu" "*.Mask")
 			(remove_unused_layers no)
-			(net 15 "3V3")
 		)
 		(pad "3" thru_hole circle
@@
 			(layers "*.Cu" "*.Mask")
 			(remove_unused_layers no)
+			(net 40 "N$35")
 		)
 		(pad "2" thru_hole circle
@@
 			(layers "*.Cu" "*.Mask")
 			(remove_unused_layers no)
+			(net 15 "3V3")
 		)
 		(pad "3" thru_hole circle
@@
 			(layers "*.Cu" "*.Mask")
 			(remove_unused_layers no)
+			(net 15 "3V3")
 		)
 		(embedded_fonts no)
@@
 			(layers "B.Cu" "B.Mask" "B.Paste")
 			(roundrect_rratio 0.25)
+			(net 44 "N$6")
 		)
 		(embedded_fonts no)
@@
 			(layers "B.Cu" "B.Mask" "B.Paste")
 			(roundrect_rratio 0.25)
+			(net 4 "N$5")
 		)
 		(embedded_fonts no)
@@
 	)
 	(gr_line
-		(start 187.065118 75.997167)
-		(end 187.065118 75.507146)
+		(start 187.082024 74.308604)
+		(end 187.082024 74.798625)
 		(stroke
 			(width 0.12)
@@
 	)
 	(gr_line
-		(start 187.453836 75.4985)
-		(end 187.065118 74.870717)
+		(start 186.693306 74.807271)
+		(end 187.082024 75.435054)
 		(stroke
 			(width 0.12)
@@
 	)
 	(gr_line
-		(start 186.670661 75.507146)
-		(end 187.065118 74.911395)
+		(start 187.476481 74.798625)
+		(end 187.082024 75.394376)
 		(stroke
 			(width 0.12)
@@
 	)
 	(gr_line
-		(start 187.065118 75.50308)
-		(end 187.45919 75.507146)
+		(start 187.082024 74.802691)
+		(end 186.687952 74.798625)
 		(stroke
 			(width 0.12)
@@
 	)
 	(gr_line
-		(start 187.065118 75.507146)
-		(end 186.670661 75.507146)
+		(start 187.082024 74.798625)
+		(end 187.476481 74.798625)
 		(stroke
 			(width 0.12)
@@
 	)
 	(gr_line
-		(start 187.574645 74.870717)
-		(end 186.55559 74.870717)
+		(start 186.572497 75.435054)
+		(end 187.591552 75.435054)
 		(stroke
 			(width 0.12)
@@
 	)
 	(gr_line
-		(start 187.065118 74.870717)
-		(end 187.065118 74.36119)
+		(start 187.082024 75.435054)
+		(end 187.082024 75.944581)
 		(stroke
 			(width 0.12)
@@
 		)
 	)
-	(gr_text "a4"
+	(gr_text "a5"
 		(at 127.899742 140.219907 0)
 		(layer "F.SilkS")
@@
 		)
 	)
+	(gr_text "+       +"
+		(at 136.928929 87.542797 0)
+		(layer "F.SilkS")
+		(effects
+			(font
+				(size 1.5 1.5)
+				(thickness 0.3)
+				(bold yes)
+			)
+			(justify left bottom)
+		)
+	)
 	(gr_text "15"
 		(at 102.500539 124.858404 270)
@@
 		(net 5)
 	)
-	(via
-		(at 173.5 73.5)
-		(size 0.7564)
-		(drill 0.35)
-		(layers "F.Cu" "B.Cu")
-		(net 5)
-	)
 	(segment
 		(start 170 76.5)
@@
 	)
 	(via
+		(at 175.26 73.66)
+		(size 0.7564)
+		(drill 0.35)
+		(layers "F.Cu" "B.Cu")
+		(net 7)
+	)
+	(via
 		(at 117.5 89.5)
 		(size 0.7564)
@@
 	)
 	(segment
-		(start 179.6161 81.343522)
-		(end 179.1081 81.8005)
-		(width 1.3716)
-		(layer "B.Cu")
-		(net 18)
-	)
-	(segment
-		(start 165.1 106.982178)
-		(end 165.1 111.76)
-		(width 1.3716)
-		(layer "B.Cu")
-		(net 18)
-	)
-	(segment
 		(start 165.1 107.5212)
 		(end 160.66 103.0812)
@@
 	)
 	(segment
-		(start 179.6161 81.343522)
-		(end 179.6796 81.229)
-		(width 1.3716)
-		(layer "B.Cu")
-		(net 18)
-	)
-	(segment
 		(start 172.7192 88.7609)
 		(end 172.7192 89.00501)
@@
 	)
 	(segment
-		(start 187.056251 77.291318)
-		(end 187.089204 77.324271)
-		(width 1.3716)
-		(layer "B.Cu")
-		(net 18)
-	)
-	(segment
 		(start 169.344393 100.197785)
 		(end 169.344393 102.737785)
@@
 	)
 	(segment
-		(start 161.331162 97.748838)
-		(end 162.56 96.52)
+		(start 152.479438 97.748838)
+		(end 148.7106 93.98)
 		(width 0.4572)
 		(layer "F.Cu")
@@
 	)
 	(segment
-		(start 148.7106 93.98)
+		(start 161.331162 97.748838)
 		(end 152.479438 97.748838)
 		(width 0.4572)
@@
 	(segment
 		(start 137.023022 85.658722)
-		(end 145.3443 93.98)
+		(end 113.147822 85.658722)
 		(width 0.4572)
 		(layer "F.Cu")
@@
 	)
 	(segment
-		(start 113.147822 85.658722)
-		(end 137.023022 85.658722)
+		(start 162.56 96.52)
+		(end 161.331162 97.748838)
 		(width 0.4572)
 		(layer "F.Cu")
@@
 	)
 	(segment
-		(start 145.3443 93.98)
-		(end 148.7106 93.98)
+		(start 148.7106 93.98)
+		(end 145.3443 93.98)
 		(width 0.4572)
 		(layer "F.Cu")
@@
 	)
 	(segment
-		(start 152.479438 97.748838)
-		(end 161.331162 97.748838)
+		(start 145.3443 93.98)
+		(end 137.023022 85.658722)
 		(width 0.4572)
 		(layer "F.Cu")
@@
 	)
 	(segment
-		(start 162.56 96.52)
-		(end 162.56 101.6)
-		(width 0.4572)
-		(layer "B.Cu")
-		(net 19)
-	)
-	(segment
 		(start 113.147822 85.658722)
 		(end 113.146878 85.658722)
@@
 	)
 	(segment
+		(start 162.56 96.52)
+		(end 162.56 101.6)
+		(width 0.4572)
+		(layer "B.Cu")
+		(net 19)
+	)
+	(segment
 		(start 111.8616 86.944)
 		(end 111.8616 91.516)
@@
 		(min_thickness 0.25)
 		(filled_areas_thickness no)
-		(fill yes
+		(fill
 			(thermal_gap 0.5)
 			(thermal_bridge_width 0.5)
@@
 		(min_thickness 0.25)
 		(filled_areas_thickness no)
-		(fill yes
+		(fill
 			(thermal_gap 0.5)
 			(thermal_bridge_width 0.5)
