File: PCB/Kicad/CENTRALE.kicad_pcb (KiCad board)
At the start: 2 copper layers, 100.3 x 72.1 mm, 77 parts, among them IC2 LM358D, J2 RJ11, J3 RJ11, U1 MCP2562-E/SN

Commit message: PCB 1.0b2
Parts:
- moved LED4 5.41 mm to (141.0, 86.0)
- moved LED2 4.73 mm to (146.1, 86.0)
- moved 7805 1.80 mm to (159.6, 108.5)
- moved GOLD_ORB_SM1 0.83 mm to (159.3, 84.2)
- renumbered LM7805 to 7805, RX2/TX2/16/17 to RX2/TX2
Routing:
- net N$33: track 92.8 -> 95.6 mm
- net VS: track 99.4 -> 101.4 mm
- net N$45: track 88.4 -> 90.4 mm
- net GND: vias 40 -> 41
Other:
- board text added: "+"
- board text added: "16 / 17"
- board text added: "1M"
- board text added: "IN"
- board text added: "OUT"
- board text added: "b2"
- board text removed: "+ +"
- board text removed: "b1"
