File: PCB/Kicad/CENTRALE.kicad_sch (KiCad schematic)
At the start: 75 parts, among them IC2 LM358D, J2 RJ11, J3 RJ11, P1 PINHD-1X4, P2 PINHD-1X4, U1 MCP2562-E{slash}SN

Commit message: PCB c3
Parts:
- removed R19: 15K, R0805, symbol CENTRALE02c3-eagle-import:R-EU_R0805
- removed SJ1, SJ2, SJ4, SJ5: SJ, SJ, symbol CENTRALE02c3-eagle-import:SJ
Other:
- moved on the sheet: D4, R18, R3

Commit message: PCB 03c4
Changed lines of the file:
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@@
 		(dnp no)
 		(property "Reference" "D1"
-			(at 203.835 225.806 0)
+			(at 203.962 227.33 0)
 			(effects
 				(font
@@
 		)
 		(property "Value" "1N5819"
-			(at 209.169 225.806 0)
+			(at 203.962 223.266 0)
 			(effects
 				(font
@@
 		(dnp no)
 		(property "Reference" "D2"
-			(at 208.915 225.806 0)
+			(at 214.376 227.33 0)
 			(effects
 				(font
@@
 		)
 		(property "Value" "1N5819"
-			(at 214.249 225.806 0)
-			(effects
-				(font
+			(at 209.55 223.012 0)
+			(effects
+				(font

Commit message: 2.10.0
Parts:
- added BoosterMode1: ~, symbol Connector_Generic:Conn_01x05
Connections:
- net at 0.96-OLED1.1 (GND), 1.3-OLED1.4, C10.1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: now also JP1.13, JP1.8, BoosterMode1.1 (Pin_1)
- net at C10.2, C5.2, D4.A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: now also BoosterMode1.5 (Pin_5)
- net at ESP32.IO14: now also JP1.11; no longer JP1.7
- net at ESP32.IO27, L6203.7 (IN2): now also BoosterMode1.4 (Pin_4); no longer JP1.8
- net at ESP32.IO32, L6203.11 (ENABLE), R10.2: now also BoosterMode1.2 (Pin_2)
- net at ESP32.IO33, L6203.5 (IN1): now also BoosterMode1.3 (Pin_3)
- net at ESP32.IO35, R20.1: now also JP1.7; no longer JP1.11

Commit message: 2.10.0 PCB production files
Parts:
- IC2: FT Rotation Offset (none) -> 270
- U1: FT Rotation Offset (none) -> -90
Changed lines of the file:
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@@
 			)
 		)
+		(property "FT Rotation Offset" "270"
+			(at 368.3 251.46 0)
+			(effects
+				(font
+					(size 1.27 1.27)
+				)
+				(hide yes)
+			)
+		)
 		(pin "1"
 		)
@@
 			)
 		)
+		(property "FT Rotation Offset" "-90"
+			(at 177.8 101.6 0)
+			(effects
+				(font
+					(size 1.27 1.27)
+				)
+				(hide yes)
+			)
+		)
 		(pin "1"
 		)
@@
 			)
 		)
+		(property "FT Rotation Offset" "270"
+			(at 322.58 218.44 0)
+			(effects
+				(font
+					(size 1.27 1.27)
+				)
+				(hide yes)
+			)
+		)
 		(pin "1"
 		)
@@
 			(at 322.58 218.44 0)
 			(effects
+				(font
+					(size 1.27 1.27)
+				)
+				(hide yes)
+			)
+		)
+		(property "FT Rotation Offset" "270"
+			(at 322.58 218.44 0)
+			(effects

Commit message: PCB 1.0 b0
Changed lines of the file:
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@@
 		(dnp no)
 		(property "Reference" "U$1"
-			(at 254 50.8 0)
+			(at 264.16 34.544 0)
 			(effects
 				(font
@@
 		)
 		(property "Value" "DC-DC-STEP-DOWN"
-			(at 254 48.26 0)
+			(at 255.016 42.926 0)
 			(effects
 				(font
@@
 		(dnp no)
 		(property "Reference" "U$4"
-			(at 248.92 76.2 0)
+			(at 259.842 60.706 0)
 			(effects
 				(font
@@
 		)
 		(property "Value" "MP1584"
-			(at 256.54 72.39 0)
-			(effects
-				(font
+			(at 257.302 68.326 0)
+			(effects
+				(font
