File: PCB/Kicad/CENTRALE.kicad_sch (KiCad schematic)
At the start: 71 parts, among them IC2 LM358D, J2 RJ11, J3 RJ11, P1 PINHD-1X4, P2 PINHD-1X4, U1 MCP2562-E{slash}SN

Commit message: PCB 1.0b2
Parts:
- added U2: L7805, symbol Regulator_Linear:L7805
- BoosterMode1: value ~ -> (none)
Connections:
- net VS: now also U2.1 (IN); no longer L6203.2 (VS)
- net at 0.96-OLED1.1 (GND), 1.3-OLED1.4, BoosterMode1.1 (Pin_1)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: now also U2.2 (GND)
- net at C4.1, C6.+, ESP32.5V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: now also U2.3 (OUT)
- new net +12V: L6203.2 (VS)
- no-connect marks 0 -> 6
Other:
- moved on the sheet: C7, R7, U$1, U$4, U1
